File: Hardware/Reference_Schematic/Advantech-Wise-1530-v1.0.0.sch (EAGLE design)
At the start: 51 parts, among them CON1 SWD-10-SMD, CON3 TE-1-1734592-0, IC1 ATECC608A, IC2 MX25R3235FM1IH0

Commit message: New Ref sch
Parts:
- removed CON1: SWD-10-SMD, mbed-HDK-Connector:SWD-10-SMD
- removed LED1: RED, mbed-HDK-Optical:SMD_LED0603
- removed MOD2: MODULE_DAUGHTER, mbed-HDK-misc-Board:MODULE_DAUGHTER
- removed R8: 1k, mbed-HDK-RLC:R0603
- removed TP1, TP2: PTR1P1-10, mbed-HDK-Test:PTR1P1-10
Connections:
- removed net PA_1: LED1.C, R8.P$2
- net +3.3V_TGT: no longer CON1.VCC, LED1.A, MOD2.3V3, TP1.TP
- net ADC0: no longer MOD2.AIN0/POT
- net ADC1: no longer MOD2.AIN1/GROVE
- net ADC2: no longer MOD2.AIN2/GROVE
- net GND: no longer CON1.GND@3, CON1.GND@5, CON1.GND@9, MOD2.GND@1, MOD2.GND@40, R8.P$1, TP2.TP
- net GPIO0: no longer MOD2.GP6/LCD-RESET
- net GPIO1: no longer MOD2.GP5/LCD-A0
- net I2C_SCL: no longer MOD2.SCL1
- net I2C_SDA: no longer MOD2.SDA1
- net I2S_CK_MCU: no longer MOD2.GP0/BUTTON
- net I2S_SD_MCU: no longer MOD2.PWM1/BLUE-LED
- net I2S_WS_MCU: no longer MOD2.PWM0/RED-LED
- net RX2: no longer MOD2.RX2
- net SPI_MISO: no longer MOD2.MISO1/LCD/SD
- net SPI_MOSI: no longer MOD2.MOSI1/LCD/SD
- net SPI_NCS0: no longer MOD2.GP7/LCD!CS
- net SPI_SCK: no longer MOD2.SCK1/LCD/SD
- net TGT_NRESET: no longer CON1.NRESET, MOD2.NRESET
- net TGT_RX: no longer CON1.NC/TDI, MOD2.TGT_RX
- net TGT_SWCLK: no longer CON1.SWCLK/TCLK, MOD2.SWCLK
- net TGT_SWDIO: no longer CON1.SWDIO/TMS, MOD2.SWDIO
- net TGT_TX: no longer CON1.KEY, MOD2.TGT_TX
- net TX2: no longer MOD2.TX2
Other:
- note added: "Advantech-WISE-1530-v1.0.0"
